File: MateLightPowerSupplyPcb.kicad_pcb (KiCad board)
At the start: 2 copper layers, 73 x 26 mm, 25 parts, among them X1 Power IN, X10 JST ZE 2, X11 JST ZE 2, X12 JST ZE 2, X13 JST ZE 2, X14 JST ZE 2, X15 JST ZE 2, X16 JST ZE 2, X17 JST ZE 2, X18 JST ZE 2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

Commit message: Added some attributes to parts
Parts:
- X1: value Power IN -> XT30U-M
- X10, X11, X12, X13, X14, X15, X16, X17, X18, X19, X20, X21, X22, X3, X4, X5, X6, X7, X8, X9: value JST ZE 2 -> S2B-ZR-SM4A-TF
- X2: value Power Out -> XT30U-M
