File: MateLightPowerSupplyPcb.kicad_sch (KiCad schematic)
At the start: 22 parts, among them X1 Power IN, X10 JST ZE 2, X11 JST ZE 2, X12 JST ZE 2, X13 JST ZE 2, X14 JST ZE 2, X15 JST ZE 2, X16 JST ZE 2, X17 JST ZE 2, X18 JST ZE 2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

Commit message: Added mounting options to PCB
Parts:
- added H1, H2, H3: MountingHole, MountingHole:MountingHole_3.2mm_M3_DIN965, symbol Mechanical:MountingHole
Changed lines of the file:
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@@
     (pin "2")
+  )
+  (symbol (lib_id "Mechanical:MountingHole") (at 229.87 97.79 0) (unit 1)
+    (in_bom yes) (on_board yes) (fields_autoplaced)
+    (property "Reference" "H2" (id 0) (at 232.41 96.9553 0)
+      (effects (font (size 1.27 1.27)) (justify left))
+    )
+    (property "Value" "MountingHole" (id 1) (at 232.41 99.4922 0)
+      (effects (font (size 1.27 1.27)) (justify left))
+    )
+    (property "Footprint" "MountingHole:MountingHole_3.2mm_M3_DIN965" (id 2) (at 229.87 97.79 0)
+      (effects (font (size 1.27 1.27)) hide)
+    )
+    (property "Datasheet" "~" (id 3) (at 229.87 97.79 0)
+      (effects (font (size 1.27 1.27)) hide)
+    )
   )
   (symbol (lib_id "Connector_Generic:Conn_01x02") (at 165.1 63.5 90) (mirror x) (unit 1)
@@
     (pin "2")
   )
+  (symbol (lib_id "Mechanical:MountingHole") (at 229.87 104.14 0) (unit 1)
+    (in_bom yes) (on_board yes) (fields_autoplaced)
+    (property "Reference" "H3" (id 0) (at 232.41 103.3053 0)
+      (effects (font (size 1.27 1.27)) (justify left))
+    )
+    (property "Value" "MountingHole" (id 1) (at 232.41 105.8422 0)
+      (effects (font (size 1.27 1.27)) (justify left))
+    )
+    (property "Footprint" "MountingHole:MountingHole_3.2mm_M3_DIN965" (id 2) (at 229.87 104.14 0)
+      (effects (font (size 1.27 1.27)) hide)
+    )
+    (property "Datasheet" "~" (id 3) (at 229.87 104.14 0)
+      (effects (font (size 1.27 1.27)) hide)
+    )
+  )
   (symbol (lib_id "Connector_Generic:Conn_01x02") (at 104.14 63.5 90) (mirror x) (unit 1)
     (in_bom yes) (on_board yes) (fields_autoplaced)
@@
     (pin "1")
   )
+  (symbol (lib_id "Mechanical:MountingHole") (at 229.87 91.44 0) (unit 1)
+    (in_bom yes) (on_board yes) (fields_autoplaced)
+    (property "Reference" "H1" (id 0) (at 232.41 90.6053 0)
+      (effects (font (size 1.27 1.27)) (justify left))
+    )
+    (property "Value" "MountingHole" (id 1) (at 232.41 93.1422 0)
+      (effects (font (size 1.27 1.27)) (justify left))
+    )
+    (property "Footprint" "MountingHole:MountingHole_3.2mm_M3_DIN965" (id 2) (at 229.87 91.44 0)
+      (effects (font (size 1.27 1.27)) hide)
+    )
+    (property "Datasheet" "~" (id 3) (at 229.87 91.44 0)
+      (effects (font (size 1.27 1.27)) hide)
+    )
+  )
   (symbol (lib_id "Connector_Generic:Conn_01x02") (at 203.2 63.5 90) (mirror x) (unit 1)
     (in_bom yes) (on_board yes) (fields_autoplaced)
@@
       (reference "#PWR0102") (unit 1) (value "GND") (footprint "")
     )
+    (path "/952b4b02-973b-4fa8-afcc-bb0d3d29c96b"
+      (reference "H1") (unit 1) (value "MountingHole") (footprint "MountingHole:MountingHole_3.2mm_M3_DIN965")
+    )
+    (path "/046e2451-9218-48fd-9037-6eb194f1771e"
+      (reference "H2") (unit 1) (value "MountingHole") (footprint "MountingHole:MountingHole_3.2mm_M3_DIN965")
+    )
+    (path "/468c19fc-049d-4b23-a555-421bdad8a190"
+      (reference "H3") (unit 1) (value "MountingHole") (footprint "MountingHole:MountingHole_3.2mm_M3_DIN965")
+    )
     (path "/67e9bfab-7e9e-44a2-9178-5c572f978806"

Commit message: Changed JST ZE to ZR connectors | added 3D models
Parts:
- X10, X11, X12, X13, X14, X15, X16, X17, X18, X19, X20, X21, X22, X3, X4, X5, X6, X7, X8, X9: footprint Connector_JST:JST_ZE_SM02B-ZESS-TB_1x02-1MP_P1.50mm_Horizontal -> h8-Connectors:JST_S2B-ZR-SM4A-TF(LF)(SN)

Commit message: Added some attributes to parts
Parts:
- H1, H2, H3: now left out of the parts list
- X1: value Power IN -> XT30U-M; LCSC# (none) -> C99101; MF (none) -> AMASS; MFN (none) -> XT30U-M; rs-online (none) -> 180-5359
- X10, X11, X12, X13, X14, X15, X16, X17, X18, X19, X20, X21, X22, X3, X4, X5, X6, X7, X8, X9: value JST ZE 2 -> S2B-ZR-SM4A-TF; LCSC# (none) -> C265329; MF (none) -> JST; MFN (none) -> S2B-ZR-SM4A-TF; digi-key (none) -> 455-1693-1-ND; rs-online (none) -> 762-0875
- X2: value Power Out -> XT30U-M; LCSC# (none) -> C99101; MF (none) -> AMASS; MFN (none) -> XT30U-M; rs-online (none) -> 180-5359

Commit message: [WIP] Added QR code and some lables to board and schematic
Changed lines of the file:
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@@
       (effects (font (size 1.27 1.27)) hide)
     )
-    (property "Datasheet" "https://jst.de/file/download/809/zh-connector" (id 3) (at 149.86 63.5 0)
+    (property "Datasheet" "~" (id 3) (at 149.86 63.5 0)
       (effects (font (size 1.27 1.27)) hide)
     )
@@
       (effects (font (size 1.27 1.27)) hide)
     )
-    (property "Datasheet" "https://jst.de/file/download/809/zh-connector" (id 3) (at 165.1 63.5 0)
+    (property "Datasheet" "~" (id 3) (at 165.1 63.5 0)
       (effects (font (size 1.27 1.27)) hide)
     )
@@
       (effects (font (size 1.27 1.27)) hide)
     )
-    (property "Datasheet" "https://static.chipdip.ru/lib/509/DOC001509847.pdf" (id 3) (at 241.3 34.29 0)
+    (property "Datasheet" "~" (id 3) (at 241.3 34.29 0)
       (effects (font (size 1.27 1.27)) hide)
     )
@@
     (pin "1")
     (pin "2")
+  )
+  (symbol (lib_id "MateLightPowerSupplyPcb-qr:QR_ProjecData") (at 25.4 186.69 0) (unit 1)
+    (in_bom no) (on_board yes) (fields_autoplaced)
+    (property "Reference" "#QR1" (id 0) (at 25.4 175.6167 0))
+    (property "Value" "QR_ProjecData" (id 1) (at 25.4 178.1536 0))
+    (property "Footprint" "QR:QR_ProjecData" (id 2) (at 25.4 197.14 0)
+      (effects (font (size 1.27 1.27)) hide)
+    )
+    (property "Datasheet" "" (id 3) (at 25.4 198.84 0)
+      (effects (font (size 1.27 1.27)) hide)
+    )
+    (property "qr_version" "2" (id 4) (at 25.4 200.54 0)
+      (effects (font (size 1.27 1.27)) hide)
+    )
+    (property "qr_size" "25" (id 5) (at 25.4 202.24 0)
+      (effects (font (size 1.27 1.27)) hide)
+    )
+    (property "qr_ecc" "1,0" (id 6) (at 25.4 203.94 0)
+      (effects (font (size 1.27 1.27)) hide)
+    )
+    (property "qr_mask" "2" (id 7) (at 25.4 205.64 0)
+      (effects (font (size 1.27 1.27)) hide)
+    )
+    (property "qr_text" "MateLightPowerSupplyPcb " (id 8) (at 25.4 207.34 0)
+      (effects (font (size 1.27 1.27)) hide)
+    )
   )
   (symbol (lib_id "Connector_Generic:Conn_01x02") (at 195.58 63.5 90) (mirror x) (unit 1)
@@
       (effects (font (size 1.27 1.27)) hide)
     )
-    (property "Datasheet" "https://jst.de/file/download/809/zh-connector" (id 3) (at 195.58 63.5 0)
+    (property "Datasheet" "~" (id 3) (at 195.58 63.5 0)
       (effects (font (size 1.27 1.27)) hide)
     )
@@
       (effects (font (size 1.27 1.27)) hide)
     )
-    (property "Datasheet" "https://jst.de/file/download/809/zh-connector" (id 3) (at 96.52 63.5 0)
+    (property "Datasheet" "~" (id 3) (at 96.52 63.5 0)
       (effects (font (size 1.27 1.27)) hide)
     )
@@
       (effects (font (size 1.27 1.27)) hide)
     )
-    (property "Datasheet" "https://jst.de/file/download/809/zh-connector" (id 3) (at 187.96 63.5 0)
+    (property "Datasheet" "~" (id 3) (at 187.96 63.5 0)
       (effects (font (size 1.27 1.27)) hide)
     )
@@
       (effects (font (size 1.27 1.27)) hide)
     )
-    (property "Datasheet" "https://jst.de/file/download/809/zh-connector" (id 3) (at 119.38 63.5 0)
+    (property "Datasheet" "~" (id 3) (at 119.38 63.5 0)
       (effects (font (size 1.27 1.27)) hide)
     )
@@
       (effects (font (size 1.27 1.27)) hide)
     )
-    (property "Datasheet" "https://jst.de/file/download/809/zh-connector" (id 3) (at 58.42 63.5 0)
+    (property "Datasheet" "~" (id 3) (at 58.42 63.5 0)
       (effects (font (size 1.27 1.27)) hide)
     )
@@
       (effects (font (size 1.27 1.27)) hide)
     )
-    (property "Datasheet" "https://jst.de/file/download/809/zh-connector" (id 3) (at 104.14 63.5 0)
+    (property "Datasheet" "~" (id 3) (at 104.14 63.5 0)
       (effects (font (size 1.27 1.27)) hide)
     )
@@
       (effects (font (size 1.27 1.27)) hide)
     )
-    (property "Datasheet" "https://jst.de/file/download/809/zh-connector" (id 3) (at 88.9 63.5 0)
+    (property "Datasheet" "~" (id 3) (at 88.9 63.5 0)
       (effects (font (size 1.27 1.27)) hide)
     )
@@
       (effects (font (size 1.27 1.27)) hide)
     )
-    (property "Datasheet" "https://jst.de/file/download/809/zh-connector" (id 3) (at 180.34 63.5 0)
+    (property "Datasheet" "~" (id 3) (at 180.34 63.5 0)
       (effects (font (size 1.27 1.27)) hide)
     )
@@
       (effects (font (size 1.27 1.27)) hide)
     )
-    (property "Datasheet" "https://static.chipdip.ru/lib/509/DOC001509847.pdf" (id 3) (at 30.48 34.29 0)
+    (property "Datasheet" "~" (id 3) (at 30.48 34.29 0)
       (effects (font (size 1.27 1.27)) hide)
     )
@@
       (effects (font (size 1.27 1.27)) hide)
     )
-    (property "Datasheet" "https://jst.de/file/download/809/zh-connector" (id 3) (at 111.76 63.5 0)
+    (property "Datasheet" "~" (id 3) (at 111.76 63.5 0)
       (effects (font (size 1.27 1.27)) hide)
     )
@@
       (effects (font (size 1.27 1.27)) hide)
     )
-    (property "Datasheet" "https://jst.de/file/download/809/zh-connector" (id 3) (at 157.48 63.5 0)
+    (property "Datasheet" "~" (id 3) (at 157.48 63.5 0)
       (effects (font (size 1.27 1.27)) hide)
     )
@@
       (effects (font (size 1.27 1.27)) hide)
     )
-    (property "Datasheet" "https://jst.de/file/download/809/zh-connector" (id 3) (at 218.44 63.5 0)
+    (property "Datasheet" "~" (id 3) (at 218.44 63.5 0)
       (effects (font (size 1.27 1.27)) hide)
     )
@@
       (effects (font (size 1.27 1.27)) hide)
     )
-    (property "Datasheet" "https://jst.de/file/download/809/zh-connector" (id 3) (at 81.28 63.5 0)
+    (property "Datasheet" "~" (id 3) (at 81.28 63.5 0)
       (effects (font (size 1.27 1.27)) hide)
     )
@@
       (effects (font (size 1.27 1.27)) hide)
     )
-    (property "Datasheet" "https://jst.de/file/download/809/zh-connector" (id 3) (at 203.2 63.5 0)
+    (property "Datasheet" "~" (id 3) (at 203.2 63.5 0)
       (effects (font (size 1.27 1.27)) hide)
     )
@@
       (effects (font (size 1.27 1.27)) hide)
     )
-    (property "Datasheet" "https://jst.de/file/download/809/zh-connector" (id 3) (at 210.82 63.5 0)
+    (property "Datasheet" "~" (id 3) (at 210.82 63.5 0)
       (effects (font (size 1.27 1.27)) hide)
     )
@@
     (pin "1")
   )
+  (symbol (lib_id "MateLightPowerSupplyPcb-qr:QR_WebUrl") (at 44.45 186.69 0) (unit 1)
+    (in_bom no) (on_board yes) (fields_autoplaced)
+    (property "Reference" "#QR2" (id 0) (at 44.375 175.6167 0))
+    (property "Value" "QR_WebUrl" (id 1) (at 44.375 178.1536 0))
+    (property "Footprint" "QR:QR_WebUrl" (id 2) (at 44.45 197.14 0)
+      (effects (font (size 1.27 1.27)) hide)
+    )
+    (property "Datasheet" "" (id 3) (at 44.45 198.84 0)
+      (effects (font (size 1.27 1.27)) hide)
+    )
+    (property "qr_version" "4" (id 4) (at 44.45 200.54 0)
+      (effects (font (size 1.27 1.27)) hide)
+    )
+    (property "qr_size" "33" (id 5) (at 44.45 202.24 0)
+      (effects (font (size 1.27 1.27)) hide)
+    )
+    (property "qr_ecc" "1,0" (id 6) (at 44.45 203.94 0)
+      (effects (font (size 1.27 1.27)) hide)
+    )
+    (property "qr_mask" "2" (id 7) (at 44.45 205.64 0)
+      (effects (font (size 1.27 1.27)) hide)
+    )
+    (property "qr_text" "https://github.com/HansAchterbahn/MateLightPowerSupplyPcb" (id 8) (at 44.45 207.34 0)
+      (effects (font (size 1.27 1.27)) hide)
+    )
+  )
   (symbol (lib_id "Connector_Generic:Conn_01x02") (at 73.66 63.5 90) (mirror x) (unit 1)
     (in_bom yes) (on_board yes) (fields_autoplaced)
@@
       (effects (font (size 1.27 1.27)) hide)
     )
-    (property "Datasheet" "https://jst.de/file/download/809/zh-connector" (id 3) (at 73.66 63.5 0)
+    (property "Datasheet" "~" (id 3) (at 73.66 63.5 0)
       (effects (font (size 1.27 1.27)) hide)
     )
@@
       (effects (font (size 1.27 1.27)) hide)
     )
-    (property "Datasheet" "https://jst.de/file/download/809/zh-connector" (id 3) (at 66.04 63.5 0)
+    (property "Datasheet" "~" (id 3) (at 66.04 63.5 0)
       (effects (font (size 1.27 1.27)) hide)
     )
@@
       (effects (font (size 1.27 1.27)) hide)
     )
-    (property "Datasheet" "https://jst.de/file/download/809/zh-connector" (id 3) (at 172.72 63.5 0)
+    (property "Datasheet" "~" (id 3) (at 172.72 63.5 0)
       (effects (font (size 1.27 1.27)) hide)
     )
@@
       (effects (font (size 1.27 1.27)) hide)
     )
-    (property "Datasheet" "https://jst.de/file/download/809/zh-connector" (id 3) (at 127 63.5 0)
+    (property "Datasheet" "~" (id 3) (at 127 63.5 0)
       (effects (font (size 1.27 1.27)) hide)
     )
@@
       (reference "#PWR0102") (unit 1) (value "GND") (footprint "")
     )
+    (path "/18081809-f203-4bae-bdda-7bd67713ea04"
+      (reference "#QR1") (unit 1) (value "QR_ProjecData") (footprint "QR:QR_ProjecData")
+    )
+    (path "/b7f5f409-1a40-4dd6-bf38-d9287db47a99"
+      (reference "#QR2") (unit 1) (value "QR_WebUrl") (footprint "QR:QR_WebUrl")
+    )
     (path "/952b4b02-973b-4fa8-afcc-bb0d3d29c96b"

Commit message: [WIP] Schematic: removed qr-code (keep on pcb), add metadata, update libraries
Parts:
- X1, X2: Manf (none) -> AMASS; Manf# (none) -> XT30U-M
- X10, X11, X12, X13, X14, X15, X16, X17, X18, X19, X20, X21, X22, X3, X4, X5, X6, X7, X8, X9: Manf (none) -> JST; Manf# (none) -> S2B-ZR-SM4A-TF
Other:
- company: (none) -> by HansAchterbahn
- title: (none) -> MateLightPowerSupply
